File: shauryapad.kicad_pcb (KiCad board)
At the start: 2 copper layers, 47.6 x 66.7 mm, 7 parts, among them SW1 SW_Push, SW2 SW_Push, SW3 SW_Push, SW4 SW_Push, U1 XIAO-RP2040-DIP

Commit message: just updating with centering or whatever fixes made
Parts:
- moved D2 6.74 mm to (188.8, 75.3)
- moved U1 1.91 mm to (171.4, 71.9)
Routing:
- net Net-(U1-GPIO1/RX): track 72.6 -> 29.4 mm
- net GND: track 110.5 -> 123.8 mm
- net Net-(U1-GPIO3/MOSI): track 43.3 -> 56.1 mm
- net Net-(D1-DOUT): track 51.2 -> 47.9 mm
- net +5V: track 36.5 -> 39.8 mm
- net Net-(D1-DIN): track 6.01 -> 8.83 mm
- net Net-(U1-GPIO4/MISO): track 47.7 -> 49.6 mm
- net Net-(U1-GPIO2/SCK): track 18.8 -> 20.3 mm
